File: hardware/kicad/Antenna-Remote.kicad_pcb (KiCad board)
At the start: 2 copper layers, 70 x 100 mm, 38 parts, among them J1 D-SUB BU 09US Female Antenna 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, J3 D-SUB ST 09US Male Ancillaries, J4 DISPLAY, K1 DIPxx-1Axx-11x, K2 DIPxx-1Axx-11x, Q1 BC550, Q2 BC550, U1 74HC164, U2 LM7805_TO220, U3 ULN2803A, U4 ESP32-DEVKITC-32D

Commit message: Hardware: document D-SUB antenna switch pinout, U3 is the TBD62783A source driver
Pin assignment of J1 follows the Amplitec RSW(4)(6)8A1R plan (positive switching, common ground on pin 3). U3 value and datasheet in schematic, board, netlist, BOM csv and BOM.xlsx changed from ULN2803A to the TBD62783A the schematic actually uses. Buzzer note names GPIO 34.
Parts:
- U3: value ULN2803A -> TBD62783A
Changed lines of the file:
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@@
 			)
 		)
-		(property "Value" "ULN2803A"
+		(property "Value" "TBD62783A"
 			(at 3.81 22.65 0)
 			(layer "F.Fab")
