File: hardware/kicad/Antenna-Remote.kicad_sch (KiCad schematic)
At the start: 38 parts, among them J1 D-SUB BU 09US Female Antenna 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, J3 D-SUB ST 09US Male Ancillaries, J4 DISPLAY, K1 CO 3570.1210.121, K2 CO 3570.1210.121, Q1 BC550, Q2 BC550, U1 74HC164, U2 LM7805_TO220, U3 ULN2803A, U4 ESP32-DEVKITC-32D

Commit message: Hardware: document D-SUB antenna switch pinout, U3 is the TBD62783A source driver
Pin assignment of J1 follows the Amplitec RSW(4)(6)8A1R plan (positive switching, common ground on pin 3). U3 value and datasheet in schematic, board, netlist, BOM csv and BOM.xlsx changed from ULN2803A to the TBD62783A the schematic actually uses. Buzzer note names GPIO 34.
Parts:
- U3: value ULN2803A -> TBD62783A
Changed lines of the file:
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@@
 			)
 		)
-		(property "Value" "ULN2803A"
+		(property "Value" "TBD62783A"
 			(at 190.1541 52.07 0)
 			(show_name no)
@@
 			)
 		)
-		(property "Datasheet" "https://www.reichelt.de/eight-darlington-arrays-dil-18-uln-2803a-p22085.html?&nbc=1"
+		(property "Datasheet" "http://toshiba.semicon-storage.com/info/docget.jsp?did=30523&prodName=TBD62783APG"
 			(at 180.34 54.61 0)
 			(hide yes)
